Commit message: add rtab sim files

File: autorally_description/urdf/autoRallyPlatform.urdf.xacro (robot description, xacro)
@@ -141,5 +141,5 @@
       <type>transmission_interface/SimpleTransmission</type>
       <joint name="${lr_prefix}_${fr_prefix}_shock">
-        <hardwareInterface>EffortJointInterface</hardwareInterface>
+        <hardwareInterface>hardware_interface/EffortJointInterface</hardwareInterface>
       </joint>
       <actuator name="${lr_prefix}_${fr_prefix}_shock_act">
@@ -168,5 +168,5 @@
       <type>transmission_interface/SimpleTransmission</type>
       <joint name="${lr_prefix}_${fr_prefix}_shock">
-        <hardwareInterface>EffortJointInterface</hardwareInterface>
+        <hardwareInterface>hardware_interface/EffortJointInterface</hardwareInterface>
       </joint>
       <actuator name="${lr_prefix}_${fr_prefix}_shock_act">
@@ -201,5 +201,5 @@
       <type>transmission_interface/SimpleTransmission</type>
       <joint name="${lr_prefix}_${fr_prefix}_axle">
-        <hardwareInterface>EffortJointInterface</hardwareInterface>
+        <hardwareInterface>hardware_interface/EffortJointInterface</hardwareInterface>
       </joint>
       <actuator name="${lr_prefix}_${fr_prefix}_axle_act">
@@ -272,5 +272,5 @@
       <type>transmission_interface/SimpleTransmission</type>
       <joint name="${lr_prefix}_steering_joint">
-        <hardwareInterface>EffortJointInterface</hardwareInterface>
+        <hardwareInterface>hardware_interface/EffortJointInterface</hardwareInterface>
       </joint>
       <actuator name="${lr_prefix}_steering_act">
@@ -396,4 +396,58 @@
       <geometry>
     <box size="0.02 0.02 0.02"/>
+      </geometry>
+    </collision>
+    <!--<visual>
+      <origin xyz="0 0 0" rpy="0 0 0"/>
+      <geometry>
+    <box size="0.02 0.02 0.02"/>
+      </geometry>
+      <material name="red"/>
+    </visual>-->
+    <inertial>
+      <mass value="1e-5" />
+      <origin xyz="0 0 0" rpy="0 0 0"/>
+      <inertia ixx="1e-6" ixy="0" ixz="0" iyy="1e-6" iyz="0" izz="1e-6" />
+    </inertial>
+  </link>
+  <joint name="left_camera_joint" type="fixed">
+    <axis xyz="0 0 -1" />
+    <origin xyz="0 -0.07 0" rpy="0 0 0"/>
+    <parent link="camera_link"/>
+    <child link="left_camera_optical_frame"/>
+  </joint>
+  <!-- Camera -->
+  <link name="left_camera_optical_frame">
+    <collision>
+      <origin xyz="0 0 0" rpy="0 0 0"/>
+      <geometry>
+    <box size="0.01 0.01 0.01"/>
+      </geometry>
+    </collision>
+    <!--<visual>
+      <origin xyz="0 0 0" rpy="0 0 0"/>
+      <geometry>
+    <box size="0.02 0.02 0.02"/>
+      </geometry>
+      <material name="red"/>
+    </visual>-->
+    <inertial>
+      <mass value="1e-5" />
+      <origin xyz="0 0 0" rpy="0 0 0"/>
+      <inertia ixx="1e-6" ixy="0" ixz="0" iyy="1e-6" iyz="0" izz="1e-6" />
+    </inertial>
+  </link>
+  <joint name="right_camera_joint" type="fixed">
+    <axis xyz="0 0 -1" />
+    <origin xyz="0 0.07 0" rpy="0 0 0"/>
+    <parent link="camera_link"/>
+    <child link="right_camera_optical_frame"/>
+  </joint>
+  <!-- Camera -->
+  <link name="right_camera_optical_frame">
+    <collision>
+      <origin xyz="0 0 0" rpy="0 0 0"/>
+      <geometry>
+    <box size="0.01 0.01 0.01"/>
       </geometry>
     </collision>
@@ -434,5 +488,5 @@
       </camera>
       <camera name="right">
-        <pose>0.02 -0.07 0 0 0 0</pose>
+        <pose>0 -0.07 0 0 0 0</pose>
         <horizontal_fov>1.3962634</horizontal_fov>
         <image>

Commit message: Changes to launch files

File: autorally_description/urdf/autoRallyPlatform.urdf.xacro (robot description, xacro)
@@ -451,58 +451,4 @@
     </inertial>
   </link>
-  <joint name="left_camera_joint" type="fixed">
-    <axis xyz="0 0 -1" />
-    <origin xyz="0 -0.07 0" rpy="0 0 0"/>
-    <parent link="camera_link"/>
-    <child link="left_camera_optical_frame"/>
-  </joint>
-  <!-- Camera -->
-  <link name="left_camera_optical_frame">
-    <collision>
-      <origin xyz="0 0 0" rpy="0 0 0"/>
-      <geometry>
-    <box size="0.01 0.01 0.01"/>
-      </geometry>
-    </collision>
-    <!--<visual>
-      <origin xyz="0 0 0" rpy="0 0 0"/>
-      <geometry>
-    <box size="0.02 0.02 0.02"/>
-      </geometry>
-      <material name="red"/>
-    </visual>-->
-    <inertial>
-      <mass value="1e-5" />
-      <origin xyz="0 0 0" rpy="0 0 0"/>
-      <inertia ixx="1e-6" ixy="0" ixz="0" iyy="1e-6" iyz="0" izz="1e-6" />
-    </inertial>
-  </link>
-  <joint name="right_camera_joint" type="fixed">
-    <axis xyz="0 0 -1" />
-    <origin xyz="0 0.07 0" rpy="0 0 0"/>
-    <parent link="camera_link"/>
-    <child link="right_camera_optical_frame"/>
-  </joint>
-  <!-- Camera -->
-  <link name="right_camera_optical_frame">
-    <collision>
-      <origin xyz="0 0 0" rpy="0 0 0"/>
-      <geometry>
-    <box size="0.01 0.01 0.01"/>
-      </geometry>
-    </collision>
-    <!--<visual>
-      <origin xyz="0 0 0" rpy="0 0 0"/>
-      <geometry>
-    <box size="0.02 0.02 0.02"/>
-      </geometry>
-      <material name="red"/>
-    </visual>-->
-    <inertial>
-      <mass value="1e-5" />
-      <origin xyz="0 0 0" rpy="0 0 0"/>
-      <inertia ixx="1e-6" ixy="0" ixz="0" iyy="1e-6" iyz="0" izz="1e-6" />
-    </inertial>
-  </link>
   <!-- camera -->
   <gazebo reference="camera_link">
@@ -528,5 +474,5 @@
       </camera>
       <camera name="right">
-        <pose>0 -0.07 0 0 0 0</pose>
+        <pose>0.02 -0.07 0 0 0 0</pose>
         <horizontal_fov>1.3962634</horizontal_fov>
         <image>
